File: Hardware/Telemetria/telemetria.brd (EAGLE design)
At the start: 100 x 80 mm, 18 parts, among them Q1 12MHz, U1 ESP-WROOM-32, U2 SN74LVC1G17-Q1_DCK_5DCK5_TEX-L, U3 SN74LVC1G17-Q1_DCK_5DCK5_TEX-L

Commit message: bmp280
Parts:
- added C10, C9: 100n, adafruit:C3216
- added C8: 100nF, adafruit:C3216
- added IC1: BMP280, bosch-bmp280:BMP280
- added J1: (no value), SparkFun-Connectors:USB-C-16P-2LAYER-PADS
- added R5, R6: 5k1, adafruit:R1206
Connections:
- new net N$10: J1.A5, R5.2
- new net N$11: J1.B5, R6.2
- new net N$7: J1.A6, J1.B6, U$1.5
- new net N$8: J1.A7, J1.B7, U$1.6
- new net N$9: C8.1, J1.SHLD1, J1.SHLD2, J1.SHLD3, J1.SHLD4
- new net SCK: IC1.4
- new net SDA: IC1.3
- net 3V3: now also C10.1, C9.1, IC1.2, IC1.6, IC1.8, J1.VBUS1, J1.VBUS2
- net GND: now also C10.2, C8.2, C9.2, IC1.1, IC1.5, IC1.7, J1.GND, J1.GND2, R5.1, R6.1

Commit message: SD e LoRa no hardware
Parts:
- added C11, C12: 100n, adafruit:C3216
- added R10, R11, R12, R13, R14, R9: 10k, adafruit:R1206
- added R7, R8: 1k, adafruit:R1206
- added U$2: LORA, lora-xl1276-8:LORAXL1276/78
- added U$3: MICROSD, adafruit:MICROSD
- BOOT: value (none) -> BOOT
- J1: value (none) -> J1
- RST: value (none) -> RST
Connections:
- new net CLK: U$2.SLCK, U1.30
- new net CMD: R10.1, U$3.3, U1.23
- new net D0: R11.1, U$3.7, U1.24
- new net D1: R12.1, U$3.8, U1.26
- new net D2: R13.1, U$3.1, U1.14
- new net D3: R14.1, U$3.2, U1.16
- new net DIO0: U$2.DIO0, U1.27
- new net GND1: C12.2
- new net LORA_CS: U$2.NSS, U1.29
- new net LORA_RST: U$2.REST, U1.28
- new net MISO: U$2.MISO, U1.31
- new net MOSI: U$2.MOSI, U1.37
- new net SD_CLK: R9.1, U$3.5, U1.13
- net 3V3: now also C11.1, C12.1, R10.2, R11.2, R12.2, R13.2, R14.2, R7.1, R8.1, R9.2, U$2.VCC, U$3.4
- net GND: now also C11.2, U$2.GND, U$2.GND1, U$2.GND2, U$3.6, U$3.MT1, U$3.MT2
- net SCK: now also R8.2, U1.36
- net SDA: now also R7.2, U1.33
