File: Hardware/Telemetria/telemetria.brd (EAGLE design)
At the start: 100 x 80 mm, 37 parts, among them IC1 BMP280, J1 J1, Q1 12MHz, U1 ESP-WROOM-32, U2 SN74LVC1G17-Q1_DCK_5DCK5_TEX-L, U3 SN74LVC1G17-Q1_DCK_5DCK5_TEX-L

Commit message: esquematico finalizado
Parts:
- removed U2, U3: SN74LVC1G17-Q1_DCK_5DCK5_TEX-L, SN74LVC1G17:DCK5_TEX-L
- added AL, SKIB_IN: (no value), con-ptr500:AK500/2-H
- added BATERIA: 3V, adafruit:CR2032-THRU
- added C13, C15: 100n, adafruit:C3216
- added C14: 22u, adafruit:C3216
- added C16, C17, CC: 1u, adafruit:C1206
- added CFF: 33n, adafruit:C1206
- added CIN: 470u, adafruit:E3,5-8
- added COUT: 680u, adafruit:E3,5-8
- added D1: BZX84-B10, diode:SOT23
- added D2: SK32, diode:SMC
- added J2: U.FL, SparkFun-Connectors:U.FL
- added L1: 47n, standardparts:0402
- added L2: 100u, inductor:INDUTOR_125125
- added Q2, Q3: IRLML6402, mosfet:SOT-23
- added R15: 10, adafruit:R1206
- added R16: 16k5, adafruit:R1206
- added R17: 10k, adafruit:R1206
- added R18: 1k, adafruit:M1206
- added R19: 1k, adafruit:R1206
- added SCHMITT-1, SCHMITT-2: SN74LVC1G17-Q1_DCK_5DCK5_TEX-L, SN74LVC1G17:DCK5_TEX-L
- added SJ1, SJ2, SJ3, SJ4, SJ5, SJ6: 0, jumper:SJ
- added U$4: NEO-M8, ubloxLib:NEO-M8
- added U$5: XL4016, XL4016:LM2576T2
- moved R14 239.1 mm to (-35.6, 82.5)
- moved R13 233.4 mm to (-30.5, 82.5)
- moved C12 232.9 mm to (-61.0, 69.8)
- moved R12 227.8 mm to (-25.4, 82.5)
- moved R11 222.4 mm to (-20.3, 82.5)
- moved R10 217.1 mm to (-15.2, 82.5)
- moved R9 205.8 mm to (-76.2, 76.2)
- moved R8 193.4 mm to (-71.1, 76.2)
- moved C11 191.2 mm to (-54.6, 69.8)
- moved R7 186.9 mm to (-66.0, 76.2)
- moved IC1 173.8 mm to (-49.5, 81.3)
- moved C10 173.3 mm to (-48.3, 69.8)
- moved C9 167.3 mm to (-41.9, 69.8)
- moved R6 163.2 mm to (-61.0, 76.2)
- moved R5 156.7 mm to (-55.9, 76.2)
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Connections:
- new net +12V: AL.1, Q2.P3
- new net +3V2: C17.1, CC.1, CIN.+, D1.3, Q2.P2, U$5.5
- new net +3V3: C16.1, C5.1, CFF.1, COUT.+, J1.VBUS1, J1.VBUS2, L2.P$2, Q3.P2, R16.1, R19.1, R2.2, R4.2, R7.1, R8.1, SCHMITT-1.5, SCHMITT-2.5, SJ1.1, SJ2.1, SJ3.2, SJ4.1, SJ5.1, SJ6.2, U$1.16, U$1.4
- new net BYPASS: CC.2, U$5.4
- new net FB: CFF.2, R16.2, R17.1, U$5.2
- new net GPS_RX: U$4.21, U1.9
- new net GPS_TX: U$4.20, U1.8
- new net N$12: BATERIA.-, U$4.24
- new net N$13: J2.FEED, L1.2, U$4.11
- new net N$14: C15.1, L1.1, R15.2
- new net N$15: R15.1, U$4.9
- new net N$16: BATERIA.+1, BATERIA.+2, U$4.22
- new net N$17: C3.1, C4.1, SJ2.2, U1.2
- new net N$18: C11.1, SJ3.1, U$2.VCC
- new net N$19: D1.1, Q2.P1, R18.2
- new net N$20: Q3.P3, SKIB_IN.2
- new net PQD: Q3.P1, R19.2
- new net SWOUT: D2.C, L2.P$1, U$5.3
- new net VDD: C12.1, R12.2, R13.2, R14.2, SJ5.2, U$3.4
- net 3V3: now also C13.1, C14.1, SJ1.2, SJ4.2, SJ6.1, U$4.23; no longer C11.1, C12.1, C3.1, C4.1, C5.1, J1.VBUS1, J1.VBUS2, R12.2, R13.2, R14.2, R2.2, R4.2, R7.1, R8.1, U$1.16, U$1.4, U$2.VCC, U$3.4, U1.2, U2.5, U3.5
- net BOOT: now also SCHMITT-1.4; no longer U2.4
- net GND: now also AL.2, C13.2, C14.2, C15.2, C16.2, C17.2, CIN.-, COUT.-, D2.A, J2.1, J2.2, R17.2, R18.1, SCHMITT-1.3, SCHMITT-2.3, SKIB_IN.1, U$4.10, U$4.12, U$4.13, U$5.1; no longer U2.3, U3.3
- net N$2: now also SCHMITT-1.2; no longer U2.2
- net N$4: now also SCHMITT-2.2; no longer U3.2
- net RST: now also SCHMITT-2.4; no longer U3.4
Routing:
- net SWOUT: track 0.00 -> 73.8 mm
- net +3V2: track 0.00 -> 59.9 mm
- net +3V3: track 0.00 -> 59.2 mm
- net FB: track 0.00 -> 23.6 mm
- net N$19: track 0.00 -> 15.6 mm
- net BYPASS: track 0.00 -> 14.0 mm
- net GND: track 0.00 -> 12.4 mm, vias 0 -> 5
- added copper zone on layer 16, net GND
Other:
- board size 100 x 80 mm -> 178.7 x 185.4 mm

Commit message: esquematico finalizado para revisao
Parts:
- added C18: 22u, adafruit:C3216
Connections:
- net GND: now also C18.2
- net N$18: now also C18.1
Changed lines of the file:
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@@
 <attribute name="VALUE" x="-77.47" y="-158.115" size="1.778" layer="27" ratio="10"/>
+</element>
+<element name="C18" library="adafruit" library_urn="urn:adsk.eagle:library:420" package="C3216" package3d_urn="urn:adsk.eagle:package:6240328/1" value="22u" x="-76.2" y="-160.02" smashed="yes">
+<attribute name="NAME" x="-77.47" y="-158.877" size="1.27" layer="25"/>
+<attribute name="VALUE" x="-77.47" y="-162.433" size="1.27" layer="27"/>
 </element>
 </elements>
@@
 <contactref element="SKIB_IN" pad="1"/>
 <contactref element="AL" pad="2"/>
+<contactref element="C18" pad="2"/>
+<wire x1="-69.8754" y1="-148.59" x2="-74.8" y2="-160.02" width="0" layer="19" extent="1-1"/>
 <wire x1="-74.9046" y1="-127" x2="-69.8754" y2="-148.59" width="0" layer="19" extent="1-1"/>
 <wire x1="-38.1" y1="-87.63" x2="-74.9046" y2="-127" width="0" layer="19" extent="1-1"/>
@@
 <contactref element="C11" pad="1"/>
 <contactref element="SJ3" pad="1"/>
+<contactref element="C18" pad="1"/>
+<wire x1="-76.962" y1="-8.89" x2="-77.6" y2="-160.02" width="0" layer="19" extent="1-1"/>
 <wire x1="-30.02" y1="40.53" x2="-76.962" y2="-8.89" width="0" layer="19" extent="1-1"/>
 <wire x1="-56.01" y1="69.85" x2="-30.02" y2="40.53" width="0" layer="19" extent="1-1"/>

Commit message: placa finalizada
Parts:
- AL: value (none) -> AL
- SKIB_IN: value (none) -> SKIB
- moved C18 340.4 mm to (168.5, 76.6), turned to 180 degrees
- moved SKIB_IN 294.7 mm to (187.7, 11.5), turned to 270 degrees
- moved Q3 293.9 mm to (178.3, 8.70), turned to 270 degrees
- moved R19 278.1 mm to (171.9, 8.80), turned to 90 degrees
- moved C15 267.6 mm to (192.3, 40.4), turned to 270 degrees
- moved SJ3 260.9 mm to (176.3, 56.9), turned to 270 degrees
- moved J2 256.1 mm to (192.3, 49.0), turned to 180 degrees
- moved L1 245.3 mm to (189.5, 47.1), turned to 180 degrees
- moved C13 239.7 mm to (169.9, 35.1), turned to 180 degrees
- moved R15 234.5 mm to (190.8, 44.6)
- moved SJ6 233.1 mm to (142.5, 56.6), turned to 180 degrees
- moved SJ1 228.7 mm to (177.3, 30.6), turned to 90 degrees
- moved AL 227.3 mm to (3.59, 65.6), turned to 90 degrees
- moved C11 223.3 mm to (168.7, 69.5), turned to 180 degrees
- moved U$4 219.2 mm to (179.8, 41.5)
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Connections:
- net N$17 renamed ESP_VCC
- net N$7 renamed USBD_P
- net N$8 renamed USBD_N
- removed net GND1: C12.2
- new net 3V3_GPS: C13.1, C14.1, SJ1.2, U$4.23
- new net SJ_3V3: C10.1, C9.1, IC1.2, IC1.6, IC1.8, SJ6.1
- net 3V3: no longer C10.1, C13.1, C14.1, C9.1, IC1.2, IC1.6, IC1.8, SJ1.2, SJ6.1, U$4.23
- net GND: now also C12.2
- net PQD: now also U1.12
Routing:
- net +3V3: track 59.2 -> 932.7 mm, vias 0 -> 3
- net GPS_TX: track 0.00 -> 137.7 mm, vias 0 -> 2
- net GPS_RX: track 0.00 -> 111.8 mm, vias 0 -> 2
- net PQD: track 0.00 -> 97.6 mm, vias 0 -> 2
- net GND: track 12.4 -> 103.7 mm, vias 5 -> 56
- net CMD: track 0.00 -> 84.9 mm, vias 0 -> 2
- net RST: track 0.00 -> 81.2 mm, vias 0 -> 2
- net D0: track 0.00 -> 78.2 mm, vias 0 -> 2
- net D3: track 0.00 -> 74.0 mm, vias 0 -> 2
- net D2: track 0.00 -> 73.9 mm, vias 0 -> 2
- net VDD: track 0.00 -> 70.3 mm
- net DIO0: track 0.00 -> 53.9 mm, vias 0 -> 2
- net MISO: track 0.00 -> 53.7 mm
- net LORA_CS: track 0.00 -> 52.4 mm
- net LORA_RST: track 0.00 -> 51.7 mm
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Other:
- board size 178.7 x 185.4 mm -> 198.6 x 80.5 mm
