File: Hardware/Telemetria/telemetria.sch (EAGLE design)
At the start: 18 parts, among them Q1 12MHz, U1 ESP-WROOM-32, U2 SN74LVC1G17-Q1_DCK_5DCK5_TEX-L, U3 SN74LVC1G17-Q1_DCK_5DCK5_TEX-L

Commit message: bmp280
Parts:
- added C10, C9: 100n, adafruit:C-USC3216
- added C8: 100nF, adafruit:C-USC3216
- added IC1: BMP280, bosch-bmp280:BMP280
- added J1: (no value), SparkFun-Connectors:USB_C_2-LAYER_PADS
- added R5, R6: 5k1, adafruit:R-US_R1206
Connections:
- new net N$10: J1.CC1, R5.2
- new net N$11: J1.CC2, R6.2
- new net N$7: J1.D+, U$1.D+
- new net N$8: J1.D-, U$1.D-
- new net N$9: C8.1, J1.SHLD
- new net SCK: IC1.SCK
- new net SDA: IC1.SDI
- net 3V3: now also C10.1, C9.1, IC1.CSB, IC1.VDD, IC1.VDDIO, J1.VBUS
- net GND: now also C10.2, C8.2, C9.2, IC1.GND, IC1.SDO, J1.GND, R5.1, R6.1
Other:
- note added: "Botões (RST + BOOT)"
- note added: "Chip ESP"
- note added: "Interface de gravação"
- moved on the sheet: C3, C4, C5, C6, C7, Q1, U1

Commit message: SD e LoRa no hardware
Parts:
- added C11, C12: 100n, adafruit:C-USC3216
- added R10, R11, R12, R13, R14, R9: 10k, adafruit:R-US_R1206
- added R7, R8: 1k, adafruit:R-US_R1206
- added U$2: LORA, lora-xl1276-8:LORA
- added U$3: MICROSD, adafruit:MICROSD
- BOOT: value (none) -> BOOT
- J1: value (none) -> J1
- RST: value (none) -> RST
Connections:
- new net CLK: U$2.SLCK, U1.IO18
- new net CMD: R10.1, U$3.DATA_IN, U1.IO15
- new net D0: R11.1, U$3.DATA_OUT, U1.IO2
- new net D1: R12.1, U$3.DAT1, U1.IO4
- new net D2: R13.1, U$3.DAT2, U1.IO12
- new net D3: R14.1, U$3.CS, U1.IO13
- new net DIO0: U$2.DIO0, U1.IO16
- new net GND1: C12.2
- new net LORA_CS: U$2.NSS, U1.IO5
- new net LORA_RST: U$2.REST, U1.IO17
- new net MISO: U$2.MISO, U1.IO19
- new net MOSI: U$2.MOSI, U1.IO23
- new net SD_CLK: R9.1, U$3.SCLK, U1.IO14
- net 3V3: now also C11.1, C12.1, R10.2, R11.2, R12.2, R13.2, R14.2, R7.1, R8.1, R9.2, U$2.VCC, U$3.VDD
- net GND: now also C11.2, U$2.GND, U$2.GND1, U$2.GND2, U$3.GND, U$3.GND1, U$3.VSS
- net SCK: now also R8.2, U1.IO22
- net SDA: now also R7.2, U1.IO21
Other:
- note added: "BMP280"
- note added: "LORA-XL1278/76"
- note added: "Socket SD/MMC"
- moved on the sheet: C10, C9, IC1
