File: Hardware/Telemetria/telemetria.sch (EAGLE design)
At the start: 37 parts, among them IC1 BMP280, J1 J1, Q1 12MHz, U1 ESP-WROOM-32, U2 SN74LVC1G17-Q1_DCK_5DCK5_TEX-L, U3 SN74LVC1G17-Q1_DCK_5DCK5_TEX-L

Commit message: circuito de gps
Parts:
- added BATERIA: 3V, adafruit:CR2032THM
- added C13, C16: 100n, adafruit:C-USC3216
- added C14: 22u, adafruit:C-USC3216
- added C15: 100p, adafruit:C-USC0805
- added J2: U.FL, SparkFun-Connectors:U.FL
- added L1: 47n, standardparts:RF-INDUCTOR.0402
- added R15: 10, adafruit:R-US_R1206
- added SJ1: (no value), jumper:SJ
- added U$4: NEO-M8, ubloxLib:NEO-M8
Connections:
- new net GPS_RX: U$4.21_RXD/SPI_MOSI
- new net GPS_TX: U$4.20_TXD/SPI_MISO
- new net N$12: BATERIA.-, U$4.24_GND
- new net N$13: J2.SIGNAL, L1.2, U$4.11_RF_IN
- new net N$14: C15.1, C16.1, L1.1, R15.2
- new net N$15: R15.1, U$4.9_VCC_RF
- new net N$16: BATERIA.+, BATERIA.+1, U$4.22_V_BCKP
- net 3V3: now also C13.1, C14.1, SJ1.1, SJ1.2, U$4.23_VCC
- net GND: now also C13.2, C14.2, C15.2, C16.2, J2.GND@0, J2.GND@1, U$4.10_GND, U$4.12_GND, U$4.13_GND
Other:
- note added: "GPS NEO-M8N"
- moved on the sheet: R10, R11, R12, R13, R14, R9

Commit message: esquematico finalizado
Parts:
- added AL, SKIB_IN: (no value), con-ptr500:AK500/2-H
- added C17, CC: 1u, adafruit:C-USC1206
- added CFF: 33n, adafruit:C-USC1206
- added CIN: 470u, adafruit:CPOL-USE3.5-8
- added COUT: 680u, adafruit:CPOL-USE3.5-8
- added D1: BZX84-B10, diode:ZENER-DIODESOT23
- added D2: SK32, diode:SCHOTTKY-DIODESMC
- added L2: 100u, inductor:INDUCTOR_125125
- added Q2, Q3: IRLML6402, mosfet:IRLML6402
- added R16: 16k5, adafruit:R-US_R1206
- added R17: 10k, adafruit:R-US_R1206
- added R18: 1k, adafruit:R-US_M1206
- added R19: 1k, adafruit:R-US_R1206
- added SJ2, SJ3, SJ4, SJ5, SJ6: 0, jumper:SJ
- added U$5: XL4016, XL4016:XL4016
- C15: value 100p -> 100n; device adafruit:C-USC0805 -> adafruit:C-USC3216
- C16: value 100n -> 1u; device adafruit:C-USC3216 -> adafruit:C-USC1206
- SJ1: value (none) -> 0
- renumbered U2 to SCHMITT-1, U3 to SCHMITT-2
Connections:
- new net +12V: AL-1.KL, Q2.D
- new net +3V2: C17.1, CC.1, CIN.+, D1.C, Q2.S, U$5.VIN
- new net +3V3: C16.1, C5.1, CFF.1, COUT.+, J1.VBUS, L2.P$2, Q3.S, R16.1, R19.1, R2.2, R4.2, R7.1, R8.1, SCHMITT-1.VCC, SCHMITT-2.VCC, SJ1.1, SJ2.1, SJ3.2, SJ4.1, SJ5.1, SJ6.2, U$1.V3, U$1.VCC
- new net BYPASS: CC.2, U$5.VC
- new net FB: CFF.2, R16.2, R17.1, U$5.FB
- new net N$17: C3.1, C4.1, SJ2.2, U1.3V3
- new net N$18: C11.1, SJ3.1, U$2.VCC
- new net N$19: D1.A, Q2.G, R18.2
- new net N$20: Q3.D, SKIB_IN-2.KL
- new net PQD: Q3.G, R19.2
- new net SWOUT: D2.C, L2.P$1, U$5.OUT
- new net VDD: C12.1, R12.2, R13.2, R14.2, SJ5.2, U$3.VDD
- net 3V3: now also SJ4.2, SJ6.1; no longer C11.1, C12.1, C3.1, C4.1, C5.1, J1.VBUS, R12.2, R13.2, R14.2, R2.2, R4.2, R7.1, R8.1, SCHMITT-1.VCC, SCHMITT-2.VCC, SJ1.1, U$1.V3, U$1.VCC, U$2.VCC, U$3.VDD, U1.3V3
- net GND: now also AL-2.KL, C17.2, CIN.-, COUT.-, D2.A, R17.2, R18.1, SKIB_IN-1.KL, U$5.GND
- net GPS_RX: now also U1.IO33
- net GPS_TX: now also U1.IO32
- net N$14: no longer C16.1
Other:
- note added: "Alimentação externa"
- note added: "Chaveamento Paraquedas"
- note added: "Conversor buck 12V para 3.3V operando em modo de condução contínua, com CI XL4016 PTH para chaveamento e MOSFET canal P na entrada para proteção contra polaridade reversa."
- note added: "Placa da telemetria do foguete de 1km para LASC 2026 (MWTH)"

Commit message: esquematico finalizado para revisao
Parts:
- added C18: 22u, adafruit:C-USC3216
Connections:
- net GND: now also C18.2
- net N$18: now also C18.1
Changed lines of the file:
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@@
 <part name="SUPPLY33" library="supply2" library_urn="urn:adsk.eagle:library:372" deviceset="GND" device=""/>
 <part name="FRAME2" library="frames" library_urn="urn:adsk.eagle:library:229" deviceset="FRAME_B_L" device=""/>
+<part name="C18" library="adafruit" library_urn="urn:adsk.eagle:library:420" deviceset="C-US" device="C3216" package3d_urn="urn:adsk.eagle:package:6240328/1" value="22u"/>
 </parts>
 <sheets>
@@
 <attribute name="DRAWING_NAME" x="269.24" y="-120.65" size="2.54" layer="94"/>
 </instance>
+<instance part="C18" gate="G$1" x="167.64" y="-12.7" smashed="yes" rot="R180">
+<attribute name="NAME" x="171.704" y="-18.415" size="1.778" layer="95" rot="R180"/>
+<attribute name="VALUE" x="166.624" y="-8.509" size="1.778" layer="96" rot="R180"/>
+</instance>
 </instances>
 <busses>
@@
 <wire x1="152.4" y1="-12.7" x2="152.4" y2="-2.54" width="0.1524" layer="91"/>
 <wire x1="152.4" y1="-2.54" x2="160.02" y2="-2.54" width="0.1524" layer="91"/>
-<wire x1="160.02" y1="-2.54" x2="170.18" y2="-2.54" width="0.1524" layer="91"/>
+<wire x1="160.02" y1="-2.54" x2="167.64" y2="-2.54" width="0.1524" layer="91"/>
+<wire x1="167.64" y1="-2.54" x2="170.18" y2="-2.54" width="0.1524" layer="91"/>
 <wire x1="160.02" y1="-7.62" x2="160.02" y2="-2.54" width="0.1524" layer="91"/>
 <junction x="160.02" y="-2.54"/>
 <pinref part="SUPPLY18" gate="GND" pin="GND"/>
+<pinref part="C18" gate="G$1" pin="2"/>
+<wire x1="167.64" y1="-2.54" x2="167.64" y2="-7.62" width="0.1524" layer="91"/>
+<junction x="167.64" y="-2.54"/>
 </segment>
 <segment>
@@
 <wire x1="160.02" y1="-17.78" x2="160.02" y2="-20.32" width="0.1524" layer="91"/>
 <junction x="160.02" y="-17.78"/>
-</segment>
-</net>
+<pinref part="C18" gate="G$1" pin="1"/>
+<wire x1="167.64" y1="-15.24" x2="167.64" y2="-17.78" width="0.1524" layer="91"/>
+<wire x1="167.64" y1="-17.78" x2="160.02" y2="-17.78" width="0.1524" layer="91"/>
+</segment>
+</net>

Commit message: placa finalizada
Parts:
- AL: value (none) -> AL
- SKIB_IN: value (none) -> SKIB
Connections:
- net N$17 renamed ESP_VCC
- net N$7 renamed USBD_P
- net N$8 renamed USBD_N
- removed net GND1: C12.2
- new net 3V3_GPS: C13.1, C14.1, SJ1.2, U$4.23_VCC
- new net SJ_3V3: C10.1, C9.1, IC1.CSB, IC1.VDD, IC1.VDDIO, SJ6.1
- net 3V3: no longer C10.1, C13.1, C14.1, C9.1, IC1.CSB, IC1.VDD, IC1.VDDIO, SJ1.2, SJ6.1, U$4.23_VCC
- net GND: now also C12.2
- net PQD: now also U1.IO27
Other:
- moved on the sheet: SJ6
