File: Hardware/Telemetria/buck_12-3v3_mcc.sch (EAGLE design)
At the start: 67 parts, among them IC1 BMP280, J1 J1, J2 U.FL, Q1 12MHz, Q2 IRLML6402, Q3 IRLML6402, U1 ESP-WROOM-32

Commit message: esquematico finalizado
Parts:
- removed BATERIA: 3V, adafruit:CR2032THM
- removed BOOT: BOOT, SparkFun-Retired:TAC_SWITCHPTH
- removed C10, C11, C12, C13, C15, C5, C9: 100n, adafruit:C-USC3216
- removed C14, C4: 22u, adafruit:C-USC3216
- removed C16, C17: 1u, adafruit:C-USC1206
- removed C2: 1u, adafruit:C-USC3216
- removed C6, C7: 22pF, adafruit:C-USC3216
- removed C8: 100nF, adafruit:C-USC3216
- removed IC1: BMP280, bosch-bmp280:BMP280
- removed J1: J1, SparkFun-Connectors:USB_C_2-LAYER_PADS
- removed J2: U.FL, SparkFun-Connectors:U.FL
- removed L2: 100u, inductor:INDUCTOR_125125
- removed Q2, Q3: IRLML6402, mosfet:IRLML6402
- removed R10, R11, R12, R13, R14, R17, R4, R9: 10k, adafruit:R-US_R1206
- removed R15: 10, adafruit:R-US_R1206
- removed R16: 16k5, adafruit:R-US_R1206
- removed R18: 1k, adafruit:R-US_M1206
- removed R19, R7, R8: 1k, adafruit:R-US_R1206
- removed R5, R6: 5k1, adafruit:R-US_R1206
- removed RST: RST, SparkFun-Retired:TAC_SWITCHPTH
- removed SCHMITT-1, SCHMITT-2: SN74LVC1G17-Q1_DCK_5DCK5_TEX-L, SN74LVC1G17:SN74LVC1G17-Q1_DCK_5DCK5_TEX-L
- removed SJ1, SJ2, SJ3, SJ4, SJ5, SJ6: 0, jumper:SJ
- removed U$2: LORA, lora-xl1276-8:LORA
- removed U$3: MICROSD, adafruit:MICROSD
- removed U$4: NEO-M8, ubloxLib:NEO-M8
- removed U$5: XL4016, XL4016:XL4016
- removed U1: ESP-WROOM-32, esp32:ESP-WROOM-32
- C1: device adafruit:C-USC3216 -> adafruit:C-USC1206
- C3: value 100n -> 1u; device adafruit:C-USC3216 -> adafruit:C-USC1206
- L1: value 47n -> 100u; device standardparts:RF-INDUCTOR.0402 -> inductor:INDUCTOR_125125
- Q1: value 12MHz -> IRLML6402; device adafruit:CRYSTALHC49S -> mosfet:IRLML6402
- R1: value 1k -> 16k5
- R3: device adafruit:R-US_R1206 -> adafruit:R-US_M1206
- U$1: value CH340G -> XL4016; device ch340g:CH340G -> XL4016:XL4016
Connections:
- removed net 3V3: C10.1, C13.1, C14.1, C9.1, IC1.CSB, IC1.VDD, IC1.VDDIO, R10.2, R11.2, R9.2, SJ1.2, SJ4.2, SJ6.1, U$4.23_VCC
- removed net BOOT: SCHMITT-1.Y, U1.IO0
- removed net CLK: U$2.SLCK, U1.IO18
- removed net CMD: R10.1, U$3.DATA_IN, U1.IO15
- removed net D0: R11.1, U$3.DATA_OUT, U1.IO2
- removed net D1: R12.1, U$3.DAT1, U1.IO4
- removed net D2: R13.1, U$3.DAT2, U1.IO12
- removed net D3: R14.1, U$3.CS, U1.IO13
- removed net DIO0: U$2.DIO0, U1.IO16
- removed net GND1: C12.2
- removed net GPS_RX: U$4.21_RXD/SPI_MOSI, U1.IO33
- removed net GPS_TX: U$4.20_TXD/SPI_MISO, U1.IO32
- removed net LORA_CS: U$2.NSS, U1.IO5
- removed net LORA_RST: U$2.REST, U1.IO17
- removed net MISO: U$2.MISO, U1.IO19
- removed net MOSI: U$2.MOSI, U1.IO23
- removed net N$1: BOOT.3, R1.1, R2.1
- removed net N$10: J1.CC1, R5.2
- removed net N$11: J1.CC2, R6.2
- removed net N$12: BATERIA.-, U$4.24_GND
- removed net N$13: J2.SIGNAL, L1.2, U$4.11_RF_IN
- removed net N$14: C15.1, L1.1, R15.2
- removed net N$15: R15.1, U$4.9_VCC_RF
- removed net N$16: BATERIA.+, BATERIA.+1, U$4.22_V_BCKP
- removed net N$17: C3.1, C4.1, SJ2.2, U1.3V3
- removed net N$18: C11.1, SJ3.1, U$2.VCC
- removed net N$19: D1.A, Q2.G, R18.2
- removed net N$2: C1.1, R1.2, SCHMITT-1.A
- removed net N$20: Q3.D
- removed net N$3: R3.1, R4.1, RST.3
- removed net N$4: C2.1, R3.2, SCHMITT-2.A
- removed net N$6: C6.1, Q1.2, U$1.XI
- removed net N$7: J1.D+, U$1.D+
- removed net N$8: J1.D-, U$1.D-
- removed net N$9: C8.1, J1.SHLD
- removed net PQD: Q3.G, R19.2
- removed net RST: SCHMITT-2.Y, U1.EN
- removed net RX0: U$1.TX, U1.RXD0
- removed net SCK: IC1.SCK, R8.2, U1.IO22
- removed net SDA: IC1.SDI, R7.2, U1.IO21
- removed net SD_CLK: R9.1, U$3.SCLK, U1.IO14
- removed net TX0: U$1.RX, U1.TXD0
- removed net VDD: C12.1, R12.2, R13.2, R14.2, SJ5.2, U$3.VDD
- net +12V: now also Q1.D; no longer Q2.D
- net +3V2: now also C3.1, Q1.S, U$1.VIN; no longer C17.1, Q2.S, U$5.VIN
- net +3V3: now also C1.1, L1.P$2, R1.1; no longer C16.1, C5.1, J1.VBUS, L2.P$2, R16.1, R19.1, R2.2, R4.2, R7.1, R8.1, SCHMITT-1.VCC, SCHMITT-2.VCC, SJ1.1, SJ2.1, SJ3.2, SJ4.1, SJ5.1, SJ6.2, U$1.V3, U$1.VCC
- net BYPASS: now also U$1.VC; no longer U$5.VC
- net FB: now also R1.2, R2.1, U$1.FB; no longer R16.2, R17.1, U$5.FB
- net GND: now also R2.2, R3.1; no longer BOOT.1, C10.2, C11.2, C13.2, C14.2, C15.2, C16.2, C17.2, C2.2, C4.2, C5.2, C6.2, C7.2, C8.2, C9.2, IC1.GND, IC1.SDO, J1.GND, J2.GND@0, J2.GND@1, R17.2, R18.1, R5.1, R6.1, RST.1, SCHMITT-1.GND, SCHMITT-2.GND, U$2.GND, U$2.GND1, U$2.GND2, U$3.GND, U$3.GND1, U$3.VSS, U$4.10_GND, U$4.12_GND, U$4.13_GND, U$5.GND, U1.GND@1, U1.GND@2, U1.GND@3, U1.GND@4
- net N$5: now also D1.A, Q1.G, R3.2; no longer C7.1, Q1.1, U$1.XO
- net SWOUT: now also L1.P$1, U$1.OUT; no longer L2.P$1, U$5.OUT
Other:
- note removed: "BMP280"
- note removed: "Botões (RST + BOOT)"
- note removed: "Chip ESP"
- note removed: "GPS NEO-M8N"
- note removed: "Interface de gravação"
- note removed: "LORA-XL1278/76"
- note removed: "Socket SD/MMC"
